Commit message: Add modular tool-changer simulation and MuJoCo viewer
Refactor the initial static lattice.urdf into a modular base + swappable tool
modules, and add an interactive MuJoCo viewer for kinematic inspection.

Tooling
- lattice_base.urdf: tool-less 5-DOF arm ending at lattice_tool_mount_link
  (carries the ConnectorPartA coupling cylinder).
- tools/{empty,gripper,screw_gripper}.xml composed onto the base by
  generate_tool_urdf.py. The tool drive servo and the ConnectorPartAcap coupling
  cap live in the tool modules (rotating tool_coupling joint in empty, locked in
  the tools), so empty is a clean bare mount.
- generated/lattice_{empty,gripper,screw_gripper}.urdf, plus lattice.urdf as the
  default gripper variant for backwards compatibility.

Viewer (mujoco_viewer.py)
- Single-window embedded workbench: offscreen MuJoCo rendered into the panel,
  grid floor, gradient sky, X/Y/Z world-axis triad, tool selector, FK sliders,
  Cartesian jog-IK with residual feedback, Zero/Wave presets, screenshot,
  fullscreen.
- Headless modes: --direct (load + IK + asset self-check), --shot,
  --contact-sheet, and a native --passive viewer.

Fixes / validation
- Mesh units: assets/so101 shells are metre-native and carry no scale; only
  ../hardware parts use scale=0.001. (Wrong mm-scaling had collapsed the so101
  shells to invisible specks.) Guarded by a degenerate-mesh preflight.
- validate_urdf.py: per-tool expected-joint sets; all three variants pass
  (single root, meshes resolve, joint limits, zero-pose FK).
- mujoco_viewer.py --direct --all-tools: all load, IK residual ~0.36 mm.

Dependencies: requirements-sim.txt adds pillow (embedded display + PNG export);
numpy ships with mujoco. The --direct self-check needs neither a display nor Pillow.

Notes: the embedded view is GPU-readback-bound (~10-15 fps on integrated GPUs;
shadows/reflections off live, on in --shot); --passive is the smooth path. The
screw_gripper is an inferred first-pass tool (see simulation/README.md).

Co-Authored-By: Claude Opus 4.8 (1M context) <noreply@anthropic.com>

File: simulation/generated/lattice_empty.urdf (robot description, URDF)
Before this commit: robot lattice_arm_gripper, 9 links, 8 joints
Links:
- removed link gripper_link
- removed link moving_jaw_so101_v1_link
- added link tool_coupling_link, mass 0.02; collision mesh filename=../../hardware/Shoulder Connector/ConnectorPartAcap.stl scale=0.001 0.001 0.001; visual mesh filename=../../hardware/Shoulder Connector/ConnectorPartAcap.stl scale=0.001 0.001 0.001
- link base_link: geometry collision mesh filename=../assets/so101/base_motor_holder_so101_v1.stl; collision mesh filename=../assets/so101/base_so101_v2.stl
- link lattice_tool_mount_link: geometry collision mesh filename=../../hardware/Shoulder Connector/ConnectorPartA.stl scale=0.001 0.001 0.001; visual mesh filename=../../hardware/Shoulder Connector/ConnectorPartA.stl scale=0.001 0.001 0.001
- link lower_arm_link: geometry collision mesh filename=../assets/so101/motor_holder_so101_wrist_v1.stl; collision mesh filename=../assets/so101/sts3215_03a_v1.stl
- link shoulder_link: geometry collision mesh filename=../assets/so101/motor_holder_so101_base_v1.stl; collision mesh filename=../assets/so101/rotation_pitch_so101_v1.stl
- link upper_arm_link: geometry collision mesh filename=../assets/so101/sts3215_03a_v1.stl; collision mesh filename=../assets/so101/upper_arm_so101_v1.stl
- link wrist_link: geometry collision mesh filename=../../hardware/Shoulder/Shoulder.stl scale=0.001 0.001 0.001; collision mesh filename=../assets/so101/sts3215_03a_no_horn_v1.stl
Joints:
- removed joint gripper
- removed joint gripper_tool_mount_joint
- added joint tool_coupling: type continuous, parent lattice_tool_mount_link, child tool_coupling_link, origin xyz=0 0 0 rpy=0 0 0, axis 0 0 1, limit effort=10 velocity=10
- joint tool0_joint: origin xyz=0.0113585558 0.0196257798 -0.0612599909 rpy=1.5708 -8.93291057e-07 0.0486831732 -> xyz=0 0 0 rpy=0 0 0; parent gripper_link -> tool_coupling_link

File: simulation/generated/lattice_gripper.urdf (robot description, URDF)
Before this commit: robot lattice_arm_gripper, 9 links, 8 joints
Links:
- link base_link: geometry collision mesh filename=../assets/so101/base_motor_holder_so101_v1.stl; collision mesh filename=../assets/so101/base_so101_v2.stl
- link gripper_link: geometry collision mesh filename=../../hardware/End Effector Connector/ConnectorPartB.stl scale=0.001 0.001 0.001; collision mesh filename=../../hardware/End Effector Connector/ConnectorPartBcap.stl scale=0.001 0.001 0.001
- link lattice_tool_mount_link: geometry collision mesh filename=../../hardware/Shoulder Connector/ConnectorPartA.stl scale=0.001 0.001 0.001; visual mesh filename=../../hardware/Shoulder Connector/ConnectorPartA.stl scale=0.001 0.001 0.001
- link lower_arm_link: geometry collision mesh filename=../assets/so101/motor_holder_so101_wrist_v1.stl; collision mesh filename=../assets/so101/sts3215_03a_v1.stl
- link moving_jaw_so101_v1_link: geometry collision mesh filename=../../hardware/End Effectors/Gripper/GripperPartb.stl scale=0.001 0.001 0.001; visual mesh filename=../../hardware/End Effectors/Gripper/GripperPartb.stl scale=0.001 0.001 0.001
- link shoulder_link: geometry collision mesh filename=../assets/so101/motor_holder_so101_base_v1.stl; collision mesh filename=../assets/so101/rotation_pitch_so101_v1.stl
- link upper_arm_link: geometry collision mesh filename=../assets/so101/sts3215_03a_v1.stl; collision mesh filename=../assets/so101/upper_arm_so101_v1.stl
- link wrist_link: geometry collision mesh filename=../../hardware/Shoulder/Shoulder.stl scale=0.001 0.001 0.001; collision mesh filename=../assets/so101/sts3215_03a_no_horn_v1.stl

File: simulation/generated/lattice_screw_gripper.urdf (robot description, URDF)
Before this commit: robot lattice_arm_gripper, 9 links, 8 joints
Links:
- removed link gripper_link
- removed link moving_jaw_so101_v1_link
- added link screw_gripper_body_link, mass 0.052; collision mesh filename=../../hardware/End Effector Connector/ConnectorPartB.stl scale=0.001 0.001 0.001; collision mesh filename=../../hardware/End Effector Connector/ConnectorPartBcap.stl scale=0.001 0.001 0.001
- added link screw_gripper_screw_link, mass 0.018; collision mesh filename=../../hardware/End Effectors/Screw Gripper/ScrewComponent.s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 scale=0.001 0.001 0.001; visual mesh filename=../../hardware/End Effectors/Screw Gripper/ScrewComponent.s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 scale=0.001 0.001 0.001
- link base_link: geometry collision mesh filename=../assets/so101/base_motor_holder_so101_v1.stl; collision mesh filename=../assets/so101/base_so101_v2.stl
- link lattice_tool_mount_link: geometry collision mesh filename=../../hardware/Shoulder Connector/ConnectorPartA.stl scale=0.001 0.001 0.001; visual mesh filename=../../hardware/Shoulder Connector/ConnectorPartA.stl scale=0.001 0.001 0.001
- link lower_arm_link: geometry collision mesh filename=../assets/so101/motor_holder_so101_wrist_v1.stl; collision mesh filename=../assets/so101/sts3215_03a_v1.stl
- link shoulder_link: geometry collision mesh filename=../assets/so101/motor_holder_so101_base_v1.stl; collision mesh filename=../assets/so101/rotation_pitch_so101_v1.stl
- link upper_arm_link: geometry collision mesh filename=../assets/so101/sts3215_03a_v1.stl; collision mesh filename=../assets/so101/upper_arm_so101_v1.stl
- link wrist_link: geometry collision mesh filename=../../hardware/Shoulder/Shoulder.stl scale=0.001 0.001 0.001; collision mesh filename=../assets/so101/sts3215_03a_no_horn_v1.stl
Joints:
- removed joint gripper
- removed joint gripper_tool_mount_joint
- added joint screw_gripper_spin: type continuous, parent screw_gripper_body_link, child screw_gripper_screw_link, origin xyz=0.0113585558 0.0196257798 -0.0612599909 rpy=-3.66884337e-06 -8.40862657e-07 0.0486831732, axis 0 1 0, limit effort=10 velocity=10
- added joint screw_gripper_tool_mount_joint: type fixed, parent lattice_tool_mount_link, child screw_gripper_body_link, origin xyz=0 0 0 rpy=0 0 0
- joint tool0_joint: origin xyz=0.0113585558 0.0196257798 -0.0612599909 rpy=1.5708 -8.93291057e-07 0.0486831732 -> xyz=0 0.048 0 rpy=0 0 0; parent gripper_link -> screw_gripper_screw_link

File: simulation/lattice_base.urdf (robot description, URDF)
Before this commit: robot lattice_arm_gripper, 9 links, 8 joints
Links:
- removed link gripper_link
- removed link moving_jaw_so101_v1_link
- removed link tool0
Joints:
- removed joint gripper
- removed joint gripper_tool_mount_joint
- removed joint tool0_joint
