Commit message: Add MuJoCo viewer and fix so101 mesh scaling in lattice.urdf
Adds an optional MuJoCo viewer for inspecting the existing lattice.urdf, and
fixes a mesh-scale bug that made the arm render as floating fragments.

mujoco_viewer.py
- Single-window embedded viewer: MuJoCo rendered offscreen straight into a dark
  Tkinter panel (one window, no stray default MuJoCo UI), on a grid floor with a
  world-axis triad. FK joint sliders, Cartesian jog buttons driven by a
  damped-least-squares IK (with residual feedback), Zero/Wave presets, live tool0
  readout, screenshot, and fullscreen.
- Headless modes (no display): --direct (load + IK + asset self-check), --shot,
  --contact-sheet, and a native --passive viewer. --urdf loads any URDF.

lattice.urdf fix
- The assets/so101/*.stl shell meshes are metre-native but were scaled by 0.001,
  collapsing them to ~0.05-0.14 mm so only the (correctly scaled) servos and
  ../hardware parts stayed visible -- the arm looked like floating fragments.
  Strips the erroneous scale from the so101 shells; ../hardware (millimetre)
  parts keep scale="0.001". The viewer's degenerate-mesh preflight guards against
  this class of error.

requirements-sim.txt: mujoco>=3.2 and pillow (embedded display + PNG export);
numpy ships with mujoco. The --direct self-check needs neither a display nor Pillow.

Verified: validate_urdf.py passes; mujoco_viewer.py --direct reports no degenerate
meshes and ~0.36 mm IK residual; offscreen renders show the assembled arm.

Note: the embedded viewport is GPU read-back bound (~10-15 fps on integrated
GPUs); --passive renders to a native GPU window for smooth navigation.

File: simulation/lattice.urdf (robot description, URDF)
Before this commit: robot lattice_so101, 9 links, 8 joints
Links:
- link base_link: geometry collision mesh filename=assets/so101/base_motor_holder_so101_v1.stl; collision mesh filename=assets/so101/base_so101_v2.stl
- link lower_arm_link: geometry collision mesh filename=assets/so101/motor_holder_so101_wrist_v1.stl; collision mesh filename=assets/so101/sts3215_03a_v1.stl
- link shoulder_link: geometry collision mesh filename=assets/so101/motor_holder_so101_base_v1.stl; collision mesh filename=assets/so101/rotation_pitch_so101_v1.stl
- link upper_arm_link: geometry collision mesh filename=assets/so101/sts3215_03a_v1.stl; collision mesh filename=assets/so101/upper_arm_so101_v1.stl
